File: HomeAudioF24.kicad_pcb (KiCad board)
At the start: 4 copper layers, 220 x 236 mm, 103 parts, among them J1 AudioJack2_Ground, J2 AD2 Connections, J3 Ardunio Conections, Q1 2N7000, Q2 TP0606, U1 LF356M, U10 LF356M, U11 LF356M, U12 LF356M, U2 LF356M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

Commit message: fixed Audio footprint
Parts:
- moved J1 10.2 mm to (235.8, 83.2), turned to 180 degrees
Routing:
- net Net-(J1-PadG): track 36.0 -> 40.6 mm
Changed lines of the file:
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@@
 	(footprint "ColorOrgan:Jack_3.5mm_Ground_RightAngle"
 		(layer "F.Cu")
-		(at 225.5275 82.9725)
+		(at 235.75 83.25 180)
 		(property "Reference" "J1"
 			(at 0 -8.5 0)
@@
 		)
 		(property "Value" "AudioJack2_Ground"
-			(at 0 12 0)
+			(at 0 12 180)
 			(unlocked yes)
 			(layer "F.Fab")
@@
 		)
 		(property "Footprint" "ColorOrgan:Jack_3.5mm_Ground_RightAngle"
-			(at 0 0 0)
+			(at 0 0 180)
 			(unlocked yes)
 			(layer "F.Fab")
@@
 		)
 		(property "Datasheet" ""
-			(at 0 0 0)
+			(at 0 0 180)
 			(unlocked yes)
 			(layer "F.Fab")
@@
 		)
 		(property "Description" "Audio Jack, 2 Poles (Mono / TS), Grounded Sleeve"
-			(at 0 0 0)
+			(at 0 0 180)
 			(unlocked yes)
 			(layer "F.Fab")
@@
 		(attr through_hole)
 		(fp_text user "${REFERENCE}"
-			(at 0 9 0)
+			(at -0.75 -6.75 180)
 			(unlocked yes)
 			(layer "F.Fab")
@@
 		)
 		(pad "G" thru_hole circle
-			(at 0 0)
+			(at 0 0 180)
 			(size 2 2)
 			(drill 1.4)
@@
 		)
 		(pad "S" thru_hole circle
-			(at 5 -5)
+			(at 5 -5 180)
 			(size 2 2)
 			(drill 1.4)
@@
 		)
 		(pad "T" thru_hole circle
-			(at 5 5)
+			(at 5 5 180)
 			(size 2 2)
 			(drill 1.4)
@@
 	)
 	(segment
-		(start 229.5275 61.9725)
-		(end 223.3775 61.9725)
+		(start 235.75 83.25)
+		(end 235.75 74.345)
 		(width 0.2)
 		(layer "F.Cu")
@@
 	)
 	(segment
-		(start 225.5275 64.1225)
+		(start 229.5275 61.9725)
 		(end 223.3775 61.9725)
 		(width 0.2)
@@
 	)
 	(segment
-		(start 225.5275 82.9725)
-		(end 225.5275 64.1225)
+		(start 229.5275 57.9725)
+		(end 229.5275 61.9725)
 		(width 0.2)
 		(layer "F.Cu")
@@
 	)
 	(segment
-		(start 229.5275 57.9725)
-		(end 229.5275 61.9725)
+		(start 235.75 74.345)
+		(end 223.3775 61.9725)
 		(width 0.2)
 		(layer "F.Cu")
