File: HomeAudioF24.kicad_pcb (KiCad board)
At the start: 4 copper layers, 220 x 90.8 mm, 103 parts, among them J1 AudioJack2_Ground, J2 AD2 Connections, J3 Ardunio Conections, Q1 2N7000, Q2 TP0606, U1 LF356M, U10 LF356M, U11 LF356M, U12 LF356M, U2 LF356M, U3 LF356M, U4 LF356M, U5 LF356M, U6 LF356M, U7 LF356M, U8 LF356M, U9 LF356M

Commit message: Added 2 logos, fixed some traces
Parts:
- added G***: LOGO, idpcoin, F.Cu at (160.5, 72.0)
- added G***: LOGOAmplab, LOGOAmplab, F.Cu at (109.0, 44.2)
- moved TP1 25.2 mm to (82.2, 44.5)
- moved G*** 18.5 mm to (137.5, 77.0)
- moved TP3 8.25 mm to (134.5, 66.8)
- moved R21 8.00 mm to (121.0, 75.0)
- moved R22 8.00 mm to (121.0, 69.0)
- moved U8 8.00 mm to (101.9, 68.0)
- moved U7 7.00 mm to (87.9, 67.9)
- moved TP2 0.25 mm to (82.5, 70.8)
- renumbered C25 to C1, C3 to C10, C4 to C11, C5 to C12, C6 to C13, C24 to C14, C23 to C15, C22 to C16, C8 to C17, C7 to C18, C10 to C19, C16 to C2, C9 to C20, C11 to C21, C12 to C22, C13 to C23, C15 to C24, C14 to C25, C18 to C3, C17 to C4, C19 to C5, C20 to C6, C21 to C7, C1 to C8, C2 to C9, D2 to D1, D1 to D2, D6 to D4, D4 to D6, J2 to J1, J1 to J2, JP2 to JP1, JP3 to JP2, JP1 to JP3, Q2 to Q1, Q1 to Q2, R4 to R1, R3 to R10, R8 to R11, R9 to R12, R29 to R13, R10 to R14, R11 to R15, R33 to R16, R32 to R17, R31 to R18, R1 to R19, R5 to R2, R14 to R20, R13 to R21, R12 to R22, R15 to R23, R16 to R24, R19 to R25, R34 to R26, R20 to R27, R21 to R28, R24 to R29, R27 to R3, R35 to R30, R18 to R31, R17 to R32, R23 to R33, R22 to R34, R26 to R35, R25 to R36, R28 to R4, R2 to R5, R7 to R6, R36 to R7, R6 to R8, R30 to R9, TP5 to TP1, TP4 to TP2, TP1 to TP3, TP6 to TP4, TP9 to TP5, TP8 to TP6, TP3 to TP8, TP2 to TP9, U4 to U1, U9 to U10, U10 to U11, U11 to U12, U5 to U2, U12 to U3, U2 to U4, U1 to U5, U3 to U6, U6 to U7, U7 to U8, U8 to U9
Routing:
- net Net-(D1-A): track 87.7 -> 62.4 mm
- net Bass_In: track 261.7 -> 278.9 mm, vias 1 -> 2
- net Net-(C3-Pad1): track 75.5 -> 60.7 mm
- net Net-(U6--IN): track 60.3 -> 66.6 mm
- net Net-(C5-Pad1): track 75.4 -> 69.1 mm
- net Net-(C7-Pad1): track 76.4 -> 82.1 mm
- net Net-(U6-OUT): track 58.9 -> 64.1 mm
- net Net-(R35-Pad1): track 27.0 -> 32.0 mm
- net Treble_Out: track 126.7 -> 131.3 mm, vias 0 -> 1
- net Net-(U7--IN): track 31.6 -> 28.4 mm
- net Net-(U1--IN): track 24.7 -> 26.4 mm
- net Modulator_Out: track 48.9 -> 50.1 mm
- net Net-(U4--IN): track 142.5 -> 141.4 mm
- net Net-(U1-OUT): track 42.1 -> 43.1 mm
- net Net-(D1-K): track 48.2 -> 48.9 mm
Other:
- board text added: "Modulator Test"
- board text added: "Shane was here"
- board text added: "SquareWave Test"
- board text added: "The AMP LAB"
- board text added: "WARNING +100°C"
- board text added: "amp-lab.org"
